Commit message: Edit files

File: sw200_description/urdf/include/sw200_v1.urdf.xacro (robot description, xacro)
@@ -10,5 +10,5 @@
   <xacro:property name="deg_to_rad" value="0.017453293" />
   <xacro:property name="sw200_base_mass" value="58.0" />
-  <xacro:property name="sw200_act_wheel_radius" value="0.09" />
+  <xacro:property name="sw200_act_wheel_radius" value="0.0625" />
   <xacro:property name="sw200_act_wheel_width" value="0.050" />
   <xacro:property name="sw200_act_wheel_mass" value="5.0" />
